File: Hardware/ADS124S08-Dev-Board/ADS124S08-Dev-Board.brd (EAGLE design)
At the start: 33 x 20.3 mm, 15 parts, among them U1 ADS124S08IPBSR

Commit message: Dev Board
Parts:
- removed GOLD_ORB_SM1: OSHWLOGOLOGO5MM, electroShri:OSHW_5MM
- removed GOLD_ORB_SM2: OSHWLOGOLOGO8MM, electroShri:OSHW_8MM
Other:
- board text removed: "https:// shridattdudhat.github.io/ ADS124S08"
- board text removed: "https://shridattdudhat.github.io/"
Changed lines of the file:
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@@
 <drawing>
 <settings>
-<setting alwaysvectorfont="no"/>
+<setting alwaysvectorfont="yes"/>
 <setting verticaltext="up"/>
 </settings>
@@
 </layers>
 <board>
-<fusionsync huburn="a.YnVzaW5lc3M6b3V0bG9vazUwMTE" projecturn="a.YnVzaW5lc3M6b3V0bG9vazUwMTEjMjAyMDA4MzEzMjc5NDEyMjY" f3durn="urn:adsk.wipprod:dm.lineage:ucpEFWP9St-Xu3qprdWjhA" pcbguid="" lastpulledtime="" lastsyncedchangeguid="" latestrevisionid="f25bfadb-3c83-4e73-b7e8-847fe77cae49" lastsyncedrevisionid="f25bfadb-3c83-4e73-b7e8-847fe77cae49" lastboardhashguid="218e1886-4eb1-b04e-ce97-630e5632baab" lastpushedtime="2020-09-16T12:36:29Z" linktopcb3d="true"/>
+<fusionsync huburn="a.YnVzaW5lc3M6b3V0bG9vazUwMTE" projecturn="a.YnVzaW5lc3M6b3V0bG9vazUwMTEjMjAyMDA4MzEzMjc5NDEyMjY" f3durn="urn:adsk.wipprod:dm.lineage:ucpEFWP9St-Xu3qprdWjhA" pcbguid="" lastpulledtime="" lastsyncedchangeguid="" latestrevisionid="f25bfadb-3c83-4e73-b7e8-847fe77cae49" lastsyncedrevisionid="f25bfadb-3c83-4e73-b7e8-847fe77cae49" lastboardhashguid="218e1886-4eb1-b04e-ce97-630e5632baab" lastpushedtime="2020-09-16T12:36:29Z" linktopcb3d="false"/>
 <plain>
 <wire x1="0" y1="0.635" x2="0" y2="19.685" width="0" layer="20"/>
@@
 <text x="29.46" y="17.77" size="0.6096" layer="22" font="vector" ratio="12" rot="MR270">AGND</text>
 <text x="32.49" y="17.16" size="0.6096" layer="22" font="vector" ratio="12" rot="MR0">GND</text>
-<text x="1.31" y="8.42" size="0.6096" layer="21" font="vector" ratio="12">ADS124S08
+<text x="32.22" y="6.39" size="0.6096" layer="21" font="vector" ratio="12" rot="R90">ADS124S08
 delta-sigma ADC
 24-bit, 4-kSPS, 12-ch</text>
-<text x="22.81" y="8.42" size="0.4064" layer="21" font="vector" ratio="12">https://shridattdudhat.github.io/</text>
-<text x="18.08" y="15.61" size="0.6096" layer="22" font="vector" ratio="12" rot="MR270">ADS124S08
-delta-sigma ADC
-24-bit, 4-kSPS, 12-ch</text>
-<text x="14.18" y="16.01" size="0.6096" layer="22" font="vector" ratio="12" rot="MR270">https://
-shridattdudhat.github.io/
-ADS124S08</text>
 </plain>
 <attributes>
@@
 <attribute name="VALUE" x="24.4923" y="13.98" size="0.4064" layer="27" ratio="10" rot="R90"/>
 </element>
-<element name="GOLD_ORB_SM1" library="electroShri" library_urn="urn:adsk.eagle:library:20683414" package="OSHW_5MM" package3d_urn="urn:adsk.eagle:package:23285996/1" value="OSHWLOGOLOGO5MM" x="27.5" y="13.3" smashed="yes"/>
-<element name="GOLD_ORB_SM2" library="electroShri" library_urn="urn:adsk.eagle:library:20683414" package="OSHW_8MM" package3d_urn="urn:adsk.eagle:package:23285995/1" value="OSHWLOGOLOGO8MM" x="27.4" y="10.6" smashed="yes" rot="MR90"/>
 </elements>
 <signals>
